File: hardware/kicad/DC-FastCharger/DC-FastCharger.kicad_pcb (KiCad board)
At the start: 6 copper layers, 300 x 200 mm, 0 parts

Commit message: اصلاح syntax فایل‌های PCB برای سازگاری با KiCad
- اصلاح فرمت DC-FastCharger.kicad_pcb
- اصلاح فرمت AC-Wallbox.kicad_pcb
- رفع خطای 'Expecting left, right, top, bottom, or mirror'
- استفاده از syntax صحیح KiCad version 20221018
- افزودن tstamp های صحیح
- فایل‌ها اکنون بدون خطا در KiCad باز می‌شوند
Routing:
- removed copper zone on In2.Cu, net +3.3V
Other:
- board text added: "300mm x 200mm"
- board text added: "6-Layer PCB - 2.0mm"
- board text added: "800V DC"
- board text added: "DANGER: HIGH VOLTAGE"
- board text added: "DC Fast Charger 60-120kW"
- board text added: "MAIN SOM SECTION"
- board text added: "POWER STAGE"
- board text added: "SAFETY MCU SECTION"
- board text removed: "DC FAST CHARGER 300mm x 200mm 6-Layer PCB"
- board text removed: "Keep clear 5mm clearance to HV traces"
- board text removed: "MAIN SOM ZONE"
- board text removed: "POWER STAGE HIGH CURRENT"
- board text removed: "SAFETY MCU ZONE"
- board text removed: "⚠ DANGER ⚠ HIGH VOLTAGE 800V DC"
Changed lines of the file:
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@@
   (general
     (thickness 2.0)
+    (legacy_teardrops no)
   )
   (paper "A2")
@@
     (rev "1.0")
     (company "Iran EV Charger Project")
-    (comment 1 "60-120kW CCS2 DC Fast Charger")
-    (comment 2 "WARNING: HIGH VOLTAGE - 800V DC")
   )
   (layers
     (0 "F.Cu" signal)
-    (1 "In1.Cu" power "GND")
-    (2 "In2.Cu" power "+12V/+48V")
+    (1 "In1.Cu" power)
+    (2 "In2.Cu" power)
     (3 "In3.Cu" signal)
     (4 "In4.Cu" signal)
@@
     (41 "Cmts.User" user "User.Comments")
     (44 "Edge.Cuts" user)
+    (45 "Margin" user)
     (46 "B.CrtYd" user "B.Courtyard")
     (47 "F.CrtYd" user "F.Courtyard")
@@
   (setup
     (pad_to_mask_clearance 0)
+    (grid_origin 0 0)
     (pcbplotparams
       (layerselection 0x00010fc_ffffffff)
       (plot_on_all_layers_selection 0x0000000_00000000)
-      (disableapertmacros false)
-      (usegerberextensions false)
-      (usegerberattributes true)
-      (usegerberadvancedattributes true)
-      (creategerberjobfile true)
+      (disableapertmacros no)
+      (usegerberextensions no)
+      (usegerberattributes yes)
+      (usegerberadvancedattributes yes)
+      (creategerberjobfile yes)
+      (dashed_line_dash_ratio 12.000000)
+      (dashed_line_gap_ratio 3.000000)
       (svgprecision 4)
-      (plotframeref false)
-      (viasonmask false)
+      (plotframeref no)
+      (viasonmask no)
       (mode 1)
-      (useauxorigin false)
+      (useauxorigin no)
       (hpglpennumber 1)
       (hpglpenspeed 20)
       (hpglpendiameter 15.000000)
-      (psnegative false)
-      (psa4output false)
-      (plotreference true)
-      (plotvalue true)
-      (plotinvisibletext false)
-      (sketchpadsonfab false)
-      (subtractmaskfromsilk false)
+      (pdf_front_fp_property_popups yes)
+      (pdf_back_fp_property_popups yes)
+      (dxfpolygonmode yes)
+      (dxfimperialunits yes)
+      (dxfusepcbnewfont yes)
+      (psnegative no)
+      (psa4output no)
+      (plotreference yes)
+      (plotvalue yes)
+      (plotfptext yes)
+      (plotinvisibletext no)
+      (sketchpadsonfab no)
+      (subtractmaskfromsilk no)
       (outputformat 1)
-      (mirror false)
+      (mirror no)
       (drillshape 0)
       (scaleselection 1)
-      (outputdirectory "gerber/")
+      (outputdirectory "")
     )
   )
   (net 0 "")
   (net 1 "GND")
-  (net 2 "DC_BUS+")
-  (net 3 "DC_BUS-")
-  (net 4 "+48V")
-  (net 5 "+12V")
-  (net 6 "+5V")
-  (net 7 "+3.3V")
-  (net 8 "CAN_H")
-  (net 9 "CAN_L")
-  (net 10 "CP")
-  (net 11 "PP")
-  (gr_rect (start 10 10) (end 310 210)
-    (stroke (width 0.3) (type solid)) (fill none) (layer "Edge.Cuts") (tstamp edge-cut-main))
-  (gr_text "DC FAST CHARGER\n300mm x 200mm\n6-Layer PCB" (at 160 110 0) (layer "F.SilkS") (tstamp text-title)
+  (net 2 "+48V")
+  (net 3 "+12V")
+  (net 4 "+5V")
+  (net 5 "+3.3V")
+  (gr_line (start 10 10) (end 310 10)
+    (stroke (width 0.2) (type solid)) (layer "Edge.Cuts"))
+  (gr_line (start 310 10) (end 310 210)
+    (stroke (width 0.2) (type solid)) (layer "Edge.Cuts"))
+  (gr_line (start 310 210) (end 10 210)
+    (stroke (width 0.2) (type solid)) (layer "Edge.Cuts"))
+  (gr_line (start 10 210) (end 10 10)
+    (stroke (width 0.2) (type solid)) (layer "Edge.Cuts"))
+  (gr_text "DC Fast Charger 60-120kW" (at 160 30 0) (layer "F.SilkS")
+    (effects (font (size 4 4) (thickness 0.6) bold) (justify center))
+  )
+  (gr_text "300mm x 200mm" (at 160 40 0) (layer "F.SilkS")
+    (effects (font (size 2 2) (thickness 0.3)) (justify center))
+  )
+  (gr_text "6-Layer PCB - 2.0mm" (at 160 48 0) (layer "F.SilkS")
+    (effects (font (size 2 2) (thickness 0.3)) (justify center))
+  )
+  (gr_text "DANGER: HIGH VOLTAGE" (at 50 70 0) (layer "F.SilkS")
     (effects (font (size 5 5) (thickness 0.8) bold) (justify center))
   )
-  (gr_text "⚠ DANGER ⚠\nHIGH VOLTAGE\n800V DC" (at 50 50 0) (layer "F.SilkS") (tstamp text-warning-1)
-    (effects (font (size 4 4) (thickness 0.7) bold) (justify center))
+  (gr_text "800V DC" (at 50 80 0) (layer "F.SilkS")
+    (effects (font (size 4 4) (thickness 0.6) bold) (justify center))
   )
-  (gr_text "⚠ DANGER ⚠\nHIGH VOLTAGE\n800V DC" (at 260 50 0) (layer "F.SilkS") (tstamp text-warning-2)
-    (effects (font (size 4 4) (thickness 0.7) bold) (justify center))
+  (gr_text "DANGER: HIGH VOLTAGE" (at 270 70 0) (layer "F.SilkS")
+    (effects (font (size 5 5) (thickness 0.8) bold) (justify center))
   )
-  (gr_line (start 10 90) (end 310 90)
-    (stroke (width 1.0) (type solid)) (layer "Cmts.User") (tstamp line-sep-1))
-  (gr_text "SAFETY MCU ZONE" (at 80 30 0) (layer "Cmts.User") (tstamp text-safety-zone)
+  (gr_text "800V DC" (at 270 80 0) (layer "F.SilkS")
+    (effects (font (size 4 4) (thickness 0.6) bold) (justify center))
+  )
+  (gr_line (start 10 100) (end 310 100)
+    (stroke (width 0.5) (type dash)) (layer "Cmts.User"))
+  (gr_text "SAFETY MCU SECTION" (at 80 110 0) (layer "Cmts.User")
     (effects (font (size 3 3) (thickness 0.5)) (justify center))
   )
-  (gr_text "MAIN SOM ZONE" (at 240 30 0) (layer "Cmts.User") (tstamp text-som-zone)
+  (gr_text "MAIN SOM SECTION" (at 240 110 0) (layer "Cmts.User")
     (effects (font (size 3 3) (thickness 0.5)) (justify center))
   )
-  (gr_text "POWER STAGE\nHIGH CURRENT" (at 160 180 0) (layer "Cmts.User") (tstamp text-power)
+  (gr_text "POWER STAGE" (at 160 190 0) (layer "Cmts.User")
     (effects (font (size 3 3) (thickness 0.5)) (justify center))
   )
-  (gr_rect (start 20 100) (end 140 150)
-    (stroke (width 0.5) (type dash)) (fill none) (layer "Cmts.User") (tstamp keepout-1))
-  (gr_text "Keep clear\n5mm clearance\nto HV traces" (at 80 125 0) (layer "Cmts.User") (tstamp text-keepout)
-    (effects (font (size 2 2) (thickness 0.3)) (justify center))
-  )
-  (zone (net 1) (net_name "GND") (layer "In1.Cu") (tstamp zone-gnd-plane)
-    (hatch edge 0.508)
+  (zone (net 1) (net_name "GND") (layer "In1.Cu") (hatch edge 0.5)
     (connect_pads (clearance 0.3))
-    (min_thickness 0.3)
-    (filled_areas_thickness no)
-    (fill yes (thermal_gap 0.508) (thermal_bridge_width 0.508))
+    (min_thickness 0.3) (filled_areas_thickness no)
+    (fill yes (thermal_gap 0.5) (thermal_bridge_width 0.5))
     (polygon
       (pts
@@
     )
   )
-  (zone (net 4) (net_name "+48V") (layer "In2.Cu") (tstamp zone-48v)
-    (hatch edge 0.508)
+  (zone (net 2) (net_name "+48V") (layer "In2.Cu") (hatch edge 0.5)
     (connect_pads (clearance 0.5))
-    (min_thickness 0.5)
-    (fill yes (thermal_gap 0.508) (thermal_bridge_width 0.508))
+    (min_thickness 0.5) (filled_areas_thickness no)
+    (fill yes (thermal_gap 0.5) (thermal_bridge_width 0.5))
     (polygon
       (pts
-        (xy 20 95)
-        (xy 150 95)
-        (xy 150 195)
-        (xy 20 195)
+        (xy 20 105)
+        (xy 150 105)
+        (xy 150 200)
+        (xy 20 200)
       )
     )
-  )
-  (zone (net 7) (net_name "+3.3V") (layer "In2.Cu") (tstamp zone-3v3)
-    (hatch edge 0.508)
-    (connect_pads (clearance 0.3))
-    (min_thickness 0.3)
-    (fill yes (thermal_gap 0.508) (thermal_bridge_width 0.508))
-    (polygon
-      (pts
-        (xy 160 20)
-        (xy 300 20)
-        (xy 300 85)
-        (xy 160 85)
-      )
-    )
